File: kolos_system_2022.kicad_pcb (KiCad board)
At the start: 4 copper layers, 125.5 x 185.3 mm, 112 parts, among them J18 8P8C_LED, J19 8P8C_LED, J29 Conn_02x05_Counter_Clockwise, J5v1 Conn_01x05_Female, K1 G5Q-1, K2 G5Q-1, K3 G5Q-1, K4 G5Q-1, K5 G5Q-1, K6 G5Q-1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

Commit message: prepared to manufacturing
Parts:
- added J1: Conn_01x01_Male, Connector_PinHeader_2.54mm:PinHeader_1x01_P2.54mm_Vertical, F.Cu at (96.3, 107.2)
- added J2: Conn_01x01_Male, Connector_PinHeader_2.54mm:PinHeader_1x01_P2.54mm_Vertical, F.Cu at (100.6, 107.2)
- moved J5v1 0.11 mm to (133.6, 181.5)
- moved Jgnd1 0.10 mm to (128.5, 191.6)
Routing:
- net Reset_in: track 0.00 -> 7.54 mm
- net Led1_in: track 0.00 -> 7.49 mm
- net  Ch6_Output: track 78.6 -> 77.8 mm
Other:
- board text added: "CH1"
- board text added: "CH2"
- board text added: "CH3"
- board text added: "CH4"
- board text added: "CH5"
- board text added: "CH6"
- board text added: "LINE"
- board text added: "Lab O-125 Moscow 2022"
- board text added: "NC1"
- board text added: "NC2"
- board text added: "NEUT"
