File: kolos_system_2022.kicad_pcb (KiCad board)
At the start: 2 copper layers, 125.5 x 185.3 mm, 129 parts, among them J1 Conn_01x01_Male, J10 Conn_01x01_Male, J11 Conn_01x01_Male, J12 Conn_01x01_Male, J13 Conn_01x01_Male, J14 Conn_01x01_Male, J15 Conn_01x01_Male, J16 Conn_01x01_Male, J17 Conn_01x01_Male, J18 8P8C_LED, J19 8P8C_LED, J2 Conn_01x01_Male, J20 Conn_01x01_Male, J21 Conn_01x01_Male, J22 Conn_01x01_Male, J23 Conn_01x01_Male, J24 Conn_01x01_Male, J25 Conn_01x01_Male, J26 Conn_01x01_Male, J27 Conn_01x01_Male, J28 Conn_01x01_Male, J29 Conn_02x05_Counter_Clockwise, J3 Conn_01x01_Male, J30 Conn_01x01_Male, J4 Conn_01x01_Male, J5 Conn_01x01_Male, J6 Conn_01x01_Male, J7 Conn_01x01_Male, J8 Conn_01x01_Male, J9 Conn_01x01_Male, K1 G5Q-1, K2 G5Q-1, K3 G5Q-1, K4 G5Q-1, K5 G5Q-1, K6 G5Q-1, Q1 BC848W, Q2 BC848W, Q3 BC848W, Q4 BC848W, Q5 BC848W, Q6 BC848W, SW1 SW_DIP_x01, U1 EL817, U2 EL817, U3 EL817, U4 EL817, U5 EL817, U6 EL817

Commit message: step 2
Parts:
- removed D12, D13, D3, D4, D5, D6: LED, LED_SMD:LED_1206_3216Metric
- removed J1, J10, J11, J12, J13, J14, J15, J16, J17, J2, J20, J21, J22, J23, J24, J25, J26, J27, J28, J3, J30, J4, J5, J6, J7, J8, J9: Conn_01x01_Male, Connector_PinHeader_2.54mm:PinHeader_1x01_P2.54mm_Vertical
- removed R1, R10, R13, R14, R15, R2, R20, R21, R22, R23, R8, R9: 1K, Resistor_SMD:R_1206_3216Metric
- added DRR1: LED, LED_SMD:LED_1206_3216Metric, F.Cu at (61.0, 74.9)
- added DRR2: LED, LED_SMD:LED_1206_3216Metric, F.Cu at (77.6, 76.2)
- added DRR3: LED, LED_SMD:LED_1206_3216Metric, F.Cu at (96.5, 76.2)
- added DRR4: LED, LED_SMD:LED_1206_3216Metric, F.Cu at (114.3, 74.9)
- added DRR5: LED, LED_SMD:LED_1206_3216Metric, F.Cu at (132.1, 74.9)
- added DRR6: LED, LED_SMD:LED_1206_3216Metric, F.Cu at (149.7, 74.9)
- added J5v1: Conn_01x05_Female, Connector_PinSocket_2.54mm:PinSocket_1x05_P2.54mm_Vertical, F.Cu at (75.7, 87.7)
- added Ja1: Conn_01x12_Male, Connector_PinSocket_2.54mm:PinSocket_1x12_P2.54mm_Vertical, F.Cu at (115.6, 97.8)
- added Ja2: Conn_01x12_Male, Connector_PinSocket_2.54mm:PinSocket_1x12_P2.54mm_Vertical, F.Cu at (90.2, 97.8)
- added Jgnd1: Conn_01x05_Female, Connector_PinSocket_2.54mm:PinSocket_1x05_P2.54mm_Vertical, F.Cu at (71.1, 87.7)
- added RR1: 1K, Resistor_SMD:R_1206_3216Metric, F.Cu at (54.6, 80.0)
- added RR2: 1K, Resistor_SMD:R_1206_3216Metric, F.Cu at (77.5, 81.3)
- added RR3: 1K, Resistor_SMD:R_1206_3216Metric, F.Cu at (90.2, 81.3)
- added RR4: 1K, Resistor_SMD:R_1206_3216Metric, F.Cu at (114.1, 80.0)
- added RR5: 1K, Resistor_SMD:R_1206_3216Metric, F.Cu at (125.0, 80.0)
- added RR6: 1K, Resistor_SMD:R_1206_3216Metric, F.Cu at (149.9, 80.0)
- added RRR1: 1K, Resistor_SMD:R_1206_3216Metric, F.Cu at (61.0, 80.0)
- added RRR2: 1K, Resistor_SMD:R_1206_3216Metric, F.Cu at (71.3, 81.3)
- added RRR3: 1K, Resistor_SMD:R_1206_3216Metric, F.Cu at (96.5, 81.3)
- added RRR4: 1K, Resistor_SMD:R_1206_3216Metric, F.Cu at (108.0, 80.0)
- added RRR5: 1K, Resistor_SMD:R_1206_3216Metric, F.Cu at (131.9, 80.0)
- added RRR6: 1K, Resistor_SMD:R_1206_3216Metric, F.Cu at (142.2, 80.0)
- K1, K2, K3, K4, K5, K6: footprint Relay_THT:Relay_SPDT_Finder_36.11 -> Chinese_emi_filter:Relay_T75
- PS1, PS2: footprint Converter_ACDC:Converter_ACDC_MeanWell_IRM-03-xx_THT -> Chinese_emi_filter:Converter_ACDC_MeanWell_IRM-03-xx_THT
- SW1: footprint Resistor_SMD:R_1206_3216Metric -> Connector_PinHeader_2.54mm:PinHeader_1x02_P2.54mm_Vertical
- moved RAIN3 203.6 mm to (153.7, 182.3)
- moved C1 198.8 mm to (120.7, 177.8), turned to -90 degrees
- moved RAIN1 197.8 mm to (138.2, 182.3)
- moved RAIN2 195.2 mm to (146.1, 182.3)
- moved R1WIRE1 179.3 mm to (132.1, 166.4), turned to -90 degrees
- moved C6 175.9 mm to (134.6, 108.0)
- moved RAIN4 173.9 mm to (139.7, 203.9)
- moved rel5-2 172.4 mm to (120.7, 39.4)
- moved R4 172.0 mm to (139.7, 119.4)
- moved Q6 172.0 mm to (149.9, 69.8)
- moved RAIN6 168.8 mm to (154.9, 203.9)
- moved D1 166.1 mm to (114.3, 153.7), turned to 90 degrees
- moved C3 164.9 mm to (120.7, 152.6), turned to 90 degrees
- moved RAIN5 162.9 mm to (147.3, 203.9)
- moved R6 162.8 mm to (139.7, 137.2)
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Connections:
- A1 pad 17: Net-(J15-Pad1) -> 3V3
- A1 pad 18: Net-(J28-Pad1) -> AREF
- A1 pad 28: Net-(J26-Pad1) -> RESET
- A1 pad 4: Net-(J14-Pad1) -> GND2
- FL1 pad 1: Net-(PS1-Pad2) -> Net-(FL1-Pad1)

Commit message: v1 of pcb
Parts:
- moved H1 119.5 mm to (159.0, 98.9)
- moved Jgnd1 118.7 mm to (128.5, 191.5), turned to 180 degrees
- moved FL1 117.4 mm to (53.2, 222.7), turned to 180 degrees
- moved J5v1 110.3 mm to (133.7, 181.5)
- moved DRR6 106.4 mm to (47.4, 46.0)
- moved Q6 105.0 mm to (46.9, 49.3), turned to 180 degrees
- moved DR6 102.3 mm to (46.5, 56.6), turned to 0 degrees
- moved rel6-2 100.5 mm to (48.1, 83.4), turned to 180 degrees
- moved rel1-2 98.5 mm to (137.7, 83.4), turned to 180 degrees
- moved RR6 98.2 mm to (57.3, 47.2), turned to 90 degrees
- moved RRR6 98.1 mm to (47.9, 53.0), turned to 180 degrees
- moved RR1 95.3 mm to (144.0, 47.1), turned to 90 degrees
- moved K6 94.6 mm to (50.3, 62.8), turned to -90 degrees
- moved U1 93.8 mm to (140.8, 46.0), turned to -90 degrees
- moved I2C-2 92.6 mm to (154.4, 184.9)
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- renumbered J18 to RS485, J19 to RS485
Connections:
- J29 pad 3: Ch1_Output ->  Ch1_Output
- J29 pad 4: Ch2_Output ->  Ch2_Output
- J29 pad 5: Ch3_Output ->  Ch3_Output
- J29 pad 6: Ch4_Output ->  Ch4_Output
- J29 pad 7: Ch5_Output ->  Ch5_Output
- J29 pad 8: Ch6_Output ->  Ch6_Output
Routing:
- net 5VA: track 0.00 -> 389.5 mm, vias 0 -> 9
- net +12V: track 0.00 -> 318.6 mm, vias 0 -> 1
- net +12VA: track 0.00 -> 315.4 mm, vias 0 -> 2
- net IN6: track 0.00 -> 301.5 mm
- net IN5: track 0.00 -> 286.5 mm
- net IN4: track 0.00 -> 269.1 mm
- net IN3: track 0.00 -> 251.7 mm
- net LINE: track 0.00 -> 247.0 mm, vias 0 -> 1
- net IN2: track 0.00 -> 233.3 mm
- net IN1: track 0.00 -> 215.0 mm
- net GND1: track 0.00 -> 164.2 mm, vias 0 -> 21
- net Net-(FL1-Pad1): track 0.00 -> 140.2 mm
- net DHT2: track 0.00 -> 120.2 mm, vias 0 -> 2
- net SCL: track 0.00 -> 112.2 mm, vias 0 -> 2
- net T/R: track 0.00 -> 104.7 mm, vias 0 -> 5
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- added copper zone on B.Cu, net GND1
- added copper zone on B.Cu, net GND2
Other:
- outline, holes or cut-outs redrawn
- board text added: "5VA"
- board text added: "DATA"
- board text added: "DHT1"
- board text added: "DHT2"
- board text added: "DIRTY LINE INPUT"
- board text added: "GND1 AREA"
- board text added: "GND2"
- board text added: "GND2_AREA"
- board text added: "RS485 cable pinout: 1 - orange+white - A 2 - orange - B 3 - green+white - NC 4 - blue - A 5 - blue+white - B 6 - green - NC 7 - brown+white - NC 8 - brown - NC"
- board text added: "SCL"
- board text added: "SDA"

Commit message: added 4 layers struct
Parts:
- removed RS485 (x2): 8P8C_LED, Connector_RJ:RJ45_Amphenol_RJHSE538X
- removed rel1-2, rel2-2, rel3-2, rel4-2, rel5-2, rel6-2: Conn_01x01_Male, Connector_PinHeader_2.54mm:PinHeader_1x01_P2.54mm_Vertical
- added J18: 8P8C_LED, Connector_RJ:RJ45_Amphenol_RJHSE538X, F.Cu at (151.0, 113.0)
- added J19: 8P8C_LED, Connector_RJ:RJ45_Amphenol_RJHSE538X, F.Cu at (151.1, 133.3)
- added rel1-NC1: Conn_01x01_Male, Connector_PinHeader_2.54mm:PinHeader_1x01_P2.54mm_Vertical, F.Cu at (140.3, 82.5)
- added rel1-NO1: Conn_01x01_Male, Connector_PinHeader_2.54mm:PinHeader_1x01_P2.54mm_Vertical, F.Cu at (131.8, 82.7)
- added rel2-NC1: Conn_01x01_Male, Connector_PinHeader_2.54mm:PinHeader_1x01_P2.54mm_Vertical, F.Cu at (126.1, 83.1)
- added rel2-NO1: Conn_01x01_Male, Connector_PinHeader_2.54mm:PinHeader_1x01_P2.54mm_Vertical, F.Cu at (114.2, 82.9)
- added rel3-NC1: Conn_01x01_Male, Connector_PinHeader_2.54mm:PinHeader_1x01_P2.54mm_Vertical, F.Cu at (107.8, 82.9)
- added rel3-NO1: Conn_01x01_Male, Connector_PinHeader_2.54mm:PinHeader_1x01_P2.54mm_Vertical, F.Cu at (95.6, 82.9)
- added rel4-NC1: Conn_01x01_Male, Connector_PinHeader_2.54mm:PinHeader_1x01_P2.54mm_Vertical, F.Cu at (88.3, 83.1)
- added rel4-NO1: Conn_01x01_Male, Connector_PinHeader_2.54mm:PinHeader_1x01_P2.54mm_Vertical, F.Cu at (78.1, 83.3)
- added rel5-NC1: Conn_01x01_Male, Connector_PinHeader_2.54mm:PinHeader_1x01_P2.54mm_Vertical, F.Cu at (60.8, 83.4)
- added rel5-NO1: Conn_01x01_Male, Connector_PinHeader_2.54mm:PinHeader_1x01_P2.54mm_Vertical, F.Cu at (72.1, 83.3)
- added rel6-NC1: Conn_01x01_Male, Connector_PinHeader_2.54mm:PinHeader_1x01_P2.54mm_Vertical, F.Cu at (52.8, 83.6)
- added rel6-NO1: Conn_01x01_Male, Connector_PinHeader_2.54mm:PinHeader_1x01_P2.54mm_Vertical, F.Cu at (44.2, 83.7)
- moved C6 7.08 mm to (134.2, 124.2)
- moved UMAX1 2.59 mm to (129.0, 124.1), turned to 0 degrees
- moved C5 1.92 mm to (136.7, 124.2), turned to 90 degrees
Routing:
- net GND1: track 164.2 -> 134.1 mm, vias 21 -> 8
- net T/R: track 104.7 -> 116.0 mm, vias 5 -> 8
- net TX: track 74.6 -> 83.9 mm, vias 0 -> 2
- net RX: track 74.4 -> 83.1 mm
- net  Ch1_Output: track 54.7 -> 62.5 mm
- net Net-(K2-Pad4): track 11.4 -> 5.95 mm
- net Net-(K6-Pad4): track 12.6 -> 7.80 mm
- net Net-(K4-Pad4): track 11.5 -> 6.87 mm
- net RS485B: track 92.5 -> 97.0 mm
- net Net-(K1-Pad4): track 11.3 -> 7.15 mm
- net Net-(K5-Pad4): track 12.1 -> 15.0 mm
- net RS485A: track 100.4 -> 103.0 mm, vias 6 -> 5
- net GND2: track 59.1 -> 61.1 mm, vias 4 -> 3
- net 5VA: track 389.5 -> 391.0 mm, vias 9 -> 10
- net IN5: track 286.5 -> 287.9 mm
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- added copper zone on In2.Cu, net +12V
- added copper zone on In2.Cu, net 5VA
- added copper zone on In1.Cu, net GND1
- added copper zone on In1.Cu, net GND2
- removed copper zone on B.Cu, net GND1
- removed copper zone on B.Cu, net GND2
Other:
- copper layers 2 -> 4

Commit message: second version of pcb
Parts:
- added J1: Conn_01x01_Male, Connector_PinHeader_2.54mm:PinHeader_1x01_P2.54mm_Vertical, F.Cu at (100.5, 107.1)
- added J2: Conn_01x01_Male, Connector_PinHeader_2.54mm:PinHeader_1x01_P2.54mm_Vertical, F.Cu at (95.8, 107.1)
Routing:
- net GND1: track 134.1 -> 155.1 mm
- net Led1_in: track 0.00 -> 7.56 mm
- net Reset_in: track 0.00 -> 7.37 mm
- net AIN2: track 72.3 -> 77.5 mm
- net AIN4: track 88.3 -> 92.2 mm
- net RS485A: track 103.0 -> 105.6 mm
- net RS485B: track 97.0 -> 94.7 mm
- net +12VA: track 315.7 -> 317.4 mm
- net GND2: track 61.1 -> 62.5 mm
- net /L3: track 33.8 -> 35.1 mm
- net SCL: track 112.2 -> 112.9 mm
Other:
- outline, holes or cut-outs redrawn
