File: kolos_system_2022.kicad_sch (KiCad schematic)
At the start: 80 parts, among them J1 Conn_01x01_Male, J10 Conn_01x01_Male, J11 Conn_01x01_Male, J12 Conn_01x01_Male, J13 Conn_01x01_Male, J14 Conn_01x01_Male, J15 Conn_01x01_Male, J16 Conn_01x01_Male, J17 Conn_01x01_Male, J18 8P8C_LED, J19 8P8C_LED, J2 Conn_01x01_Male, J20 Conn_01x01_Male, J21 Conn_01x01_Male, J22 Conn_01x01_Male, J23 Conn_01x01_Male, J24 Conn_01x01_Male, J25 Conn_01x01_Male, J26 Conn_02x05_Counter_Clockwise, J3 Conn_01x01_Male, J4 Conn_01x01_Male, J5 Conn_01x01_Male, J6 Conn_01x01_Male, J7 Conn_01x01_Male, J8 Conn_01x01_Male, J9 Conn_01x01_Male, K1 G5Q-1, K2 G5Q-1, K3 G5Q-1, K4 G5Q-1, Q1 BC848W, Q2 BC848W, Q3 BC848W, Q4 BC848W, SW1 SW_DIP_x01, U1 EL817, U2 EL817, U3 EL817, U4 EL817, U5 MAX485E

Commit message: new
Parts:
- A1: footprint Module:Arduino_UNO_R3 -> Module:Arduino_Nano
Changed lines of the file:
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@@
       (effects (font (size 1.27 1.27)) (justify left))
     )
-    (property "Footprint" "Module:Arduino_UNO_R3" (id 2) (at 58.42 116.84 0)
+    (property "Footprint" "Module:Arduino_Nano" (id 2) (at 58.42 116.84 0)
       (effects (font (size 1.27 1.27) italic) hide)
     )
@@
     )
     (path "/f6352f69-fb16-4200-81dd-ca1d356a2aaf"
-      (reference "A1") (unit 1) (value "Arduino_UNO_R3") (footprint "Module:Arduino_UNO_R3")
+      (reference "A1") (unit 1) (value "Arduino_UNO_R3") (footprint "Module:Arduino_Nano")
     )
     (path "/a7972806-b76a-4096-8493-49e7e1165a91"

Commit message: fuuu
Parts:
- removed J26: Conn_02x05_Counter_Clockwise, Connector_Molex:Molex_Mini-Fit_Jr_5566-10A_2x05_P4.20mm_Vertical, symbol Connector_Generic:Conn_02x05_Counter_Clockwise
- added 1WIRE1, 1WIRE2, 1WIRE3, DHT_1, DHT_2: Conn_01x03, symbol Connector_Generic:Conn_01x03
- added AIN_1, AIN_2, AIN_3, AIN_4: Conn_01x02, symbol Connector_Generic:Conn_01x02
- added D12, D13: LED, LED_SMD:LED_1206_3216Metric, symbol Device:LED
- added D14, D15: DIODE, Diode_THT:D_A-405_P7.62mm_Horizontal, symbol pspice:DIODE
- added I2C-1, I2C-2, I2C-3: Conn_01x04, symbol Connector_Generic:Conn_01x04
- added J26, J27, J28, rel1-2, rel2-2, rel3-2, rel4-2, rel5-2, rel6-2: Conn_01x01_Male, Connector_PinHeader_2.54mm:PinHeader_1x01_P2.54mm_Vertical, symbol Connector:Conn_01x01_Male
- added J29: Conn_02x06_Counter_Clockwise, symbol Connector_Generic:Conn_02x06_Counter_Clockwise
- added K5, K6: G5Q-1, Relay_THT:Relay_SPDT_Omron-G5Q-1, symbol Relay:G5Q-1
- added Q5, Q6: BC848W, Package_TO_SOT_SMD:SOT-323_SC-70, symbol Transistor_BJT:BC848W
- added R1WIRE1: 4.7K, Resistor_SMD:R_1206_3216Metric, symbol Device:R
- added R20, R21, R22, R23: 1K, Resistor_SMD:R_1206_3216Metric, symbol Device:R
- added RAIN1, RAIN2, RAIN3, RAIN4: 10K, Resistor_SMD:R_1206_3216Metric, symbol Device:R
- added U6, U7: EL817, Package_DIP:DIP-4_W7.62mm, symbol Isolator:EL817
- C2, C4: footprint (none) -> Capacitor_THT:CP_Radial_D8.0mm_P2.50mm
Connections:
- net +12V: now also D14.2 (A), D15.2 (A), K5.5, K6.5, U6.4, U7.4
- net +12VA: now also R20.1, R21.1
- net 5VA: now also 1WIRE1.1 (Pin_1), 1WIRE2.1 (Pin_1), 1WIRE3.1 (Pin_1), DHT_1.1 (Pin_1), DHT_2.1 (Pin_1), I2C-1.3 (Pin_3), I2C-2.3 (Pin_3), I2C-3.3 (Pin_3), R1WIRE1.1, RAIN1.2, RAIN2.2, RAIN3.2, RAIN4.2
- net Ch1_Output: now also J29.3 (Pin_3)
- net Ch2_Output: now also J29.4 (Pin_4)
- net Ch3_Output: now also J29.5 (Pin_5)
- net Ch4_Output: now also J29.6 (Pin_6)
- net GND1: now also Q5.2 (E), Q6.2 (E)
- net GND2: now also 1WIRE1.3 (Pin_3), 1WIRE2.3 (Pin_3), 1WIRE3.3 (Pin_3), AIN_1.2 (Pin_2), AIN_2.2 (Pin_2), AIN_3.2 (Pin_2), AIN_4.2 (Pin_2), DHT_1.3 (Pin_3), DHT_2.3 (Pin_3), I2C-1.4 (Pin_4), I2C-2.4 (Pin_4), I2C-3.4 (Pin_4)
- net LINE: now also J29.1 (Pin_1), K5.2, K6.2
- net Led1_in: now also J29.10 (Pin_10)
- net Led2_in: now also J29.11 (Pin_11)
- net NEUT: now also J29.2 (Pin_2)
- net Reset_in: now also J29.12 (Pin_12)
- net IN6: now reaches A1.22 (D7), J6.1 (Pin_1)
- net IN6: now also D13.1 (K)
- net AIN4: now reaches A1.12 (A3), J23.1 (Pin_1)
- net AIN4: now also AIN_4.1 (Pin_1), RAIN4.1
- net at K4.4: now also rel4-2.1 (Pin_1)
- net at K2.4: now also rel2-2.1 (Pin_1)
- net 1WIRE_DATA: now reaches A1.23 (D8), J7.1 (Pin_1)
- net 1WIRE_DATA: now also 1WIRE1.2 (Pin_2), 1WIRE2.2 (Pin_2), 1WIRE3.2 (Pin_2), R1WIRE1.2
- net SCL: now reaches A1.14 (SCL/A5), J25.1 (Pin_1)
- net SCL: now also I2C-1.1 (Pin_1), I2C-2.1 (Pin_1), I2C-3.1 (Pin_1)
- net AIN3: now reaches A1.11 (A2), J22.1 (Pin_1)
- net AIN3: now also AIN_3.1 (Pin_1), RAIN3.1
- net AIN2: now reaches A1.10 (A1), J21.1 (Pin_1)
- net AIN2: now also AIN_2.1 (Pin_1), RAIN2.1
- net IN5: now reaches A1.21 (D6), J5.1 (Pin_1)
- net IN5: now also D12.1 (K)
- net at K1.4: now also rel1-2.1 (Pin_1)
- net at K3.4: now also rel3-2.1 (Pin_1)
- net DHT1: now reaches A1.27 (D12), J11.1 (Pin_1)
- net DHT1: now also DHT_1.2 (Pin_2)
- net SDA: now reaches A1.13 (SDA/A4), J24.1 (Pin_1)
- net SDA: now also I2C-1.2 (Pin_2), I2C-2.2 (Pin_2), I2C-3.2 (Pin_2)
- net DHT2: now reaches A1.28 (D13), J12.1 (Pin_1)
- net DHT2: now also DHT_2.2 (Pin_2)
- net at A1.2 (IOREF): now also J27.1 (Pin_1)
- net at A1.3 (~{RESET}): now also J26.1 (Pin_1)
- net at A1.30 (AREF): now also J28.1 (Pin_1)
- net AIN1: now reaches A1.9 (A0), J20.1 (Pin_1)
- net AIN1: now also AIN_1.1 (Pin_1), RAIN1.1
- new net: K5.4, rel5-2.1 (Pin_1)
- new net: D15.1 (K), K6.1, Q6.3 (C)
- new net: R22.1, U6.3
- new net: Q5.1 (B), R22.2
- new net: R23.1, U7.3
- new net: Q6.1 (B), R23.2
- new net: K6.4, rel6-2.1 (Pin_1)
- new net: R20.2, U6.1
- new net: D14.1 (K), K5.1, Q5.3 (C)
- new net: R21.2, U7.1
- new net: D12.2 (A), U6.2
- new net: D13.2 (A), U7.2
- new net  Ch5_Output: K5.3
- new net  Ch6_Output: K6.3
- new net Ch5_Output: J29.8 (Pin_8)
- new net Ch6_Output: J29.7 (Pin_7)
- no-connect marks 7 -> 6
Other:
- note added: "1-WIRE pins"
- note added: "Analog/Button input pins"
- note added: "DHT pins"
- note added: "I2C pins"
- note added: "to device cover"
- moved on the sheet: D4, D9, J2, K2, Q2, R13, R8, U2

Commit message: holes
Parts:
- added H? (x4): MountingHole, symbol Mechanical:MountingHole
Changed lines of the file:
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@@
     (pin "2")
+  )
+  (symbol (lib_id "Mechanical:MountingHole") (at 391.16 209.55 0) (unit 1)
+    (in_bom yes) (on_board yes) (fields_autoplaced)
+    (property "Reference" "H?" (id 0) (at 393.7 208.2799 0)
+      (effects (font (size 1.27 1.27)) (justify left) hide)
+    )
+    (property "Value" "MountingHole" (id 1) (at 393.7 210.8199 0)
+      (effects (font (size 1.27 1.27)) (justify left) hide)
+    )
+    (property "Footprint" "" (id 2) (at 391.16 209.55 0)
+      (effects (font (size 1.27 1.27)) hide)
+    )
+    (property "Datasheet" "~" (id 3) (at 391.16 209.55 0)
+      (effects (font (size 1.27 1.27)) hide)
+    )
   )
   (symbol (lib_id "Converter_ACDC:VTX-214-010-112") (at 66.04 31.75 0) (unit 1)
@@
     (pin "9")
   )
+  (symbol (lib_id "Mechanical:MountingHole") (at 391.16 215.9 0) (unit 1)
+    (in_bom yes) (on_board yes) (fields_autoplaced)
+    (property "Reference" "H?" (id 0) (at 393.7 214.6299 0)
+      (effects (font (size 1.27 1.27)) (justify left) hide)
+    )
+    (property "Value" "MountingHole" (id 1) (at 393.7 217.1699 0)
+      (effects (font (size 1.27 1.27)) (justify left) hide)
+    )
+    (property "Footprint" "" (id 2) (at 391.16 215.9 0)
+      (effects (font (size 1.27 1.27)) hide)
+    )
+    (property "Datasheet" "~" (id 3) (at 391.16 215.9 0)
+      (effects (font (size 1.27 1.27)) hide)
+    )
+  )
   (symbol (lib_id "power:LINE") (at 256.54 179.07 0) (unit 1)
     (in_bom yes) (on_board yes) (fields_autoplaced)
@@
     )
     (pin "1")
+  )
+  (symbol (lib_id "Mechanical:MountingHole") (at 391.16 222.25 0) (unit 1)
+    (in_bom yes) (on_board yes) (fields_autoplaced)
+    (property "Reference" "H?" (id 0) (at 393.7 220.9799 0)
+      (effects (font (size 1.27 1.27)) (justify left) hide)
+    )
+    (property "Value" "MountingHole" (id 1) (at 393.7 223.5199 0)
+      (effects (font (size 1.27 1.27)) (justify left) hide)
+    )
+    (property "Footprint" "" (id 2) (at 391.16 222.25 0)
+      (effects (font (size 1.27 1.27)) hide)
+    )
+    (property "Datasheet" "~" (id 3) (at 391.16 222.25 0)
+      (effects (font (size 1.27 1.27)) hide)
+    )
   )
   (symbol (lib_id "Connector:Conn_01x01_Male") (at 80.01 111.76 180) (unit 1)
@@
     (pin "1")
   )
+  (symbol (lib_id "Mechanical:MountingHole") (at 391.16 228.6 0) (unit 1)
+    (in_bom yes) (on_board yes) (fields_autoplaced)
+    (property "Reference" "H?" (id 0) (at 393.7 227.3299 0)
+      (effects (font (size 1.27 1.27)) (justify left) hide)
+    )
+    (property "Value" "MountingHole" (id 1) (at 393.7 229.8699 0)
+      (effects (font (size 1.27 1.27)) (justify left) hide)
+    )
+    (property "Footprint" "" (id 2) (at 391.16 228.6 0)
+      (effects (font (size 1.27 1.27)) hide)
+    )
+    (property "Datasheet" "~" (id 3) (at 391.16 228.6 0)
+      (effects (font (size 1.27 1.27)) hide)
+    )
+  )
   (symbol (lib_id "Device:R") (at 210.82 243.84 90) (unit 1)
     (in_bom yes) (on_board yes) (fields_autoplaced)
@@
       (reference "FL1") (unit 1) (value "Filter_EMI") (footprint "")
     )
+    (path "/0802365f-ed99-42a1-9d8b-c19e4eb495ec"
+      (reference "H?") (unit 1) (value "MountingHole") (footprint "")
+    )
+    (path "/592172b8-b84d-438d-998a-358c5f4a4bed"
+      (reference "H?") (unit 1) (value "MountingHole") (footprint "")
+    )
+    (path "/e1a83c4a-6406-4978-a086-5a79f3e22a48"
+      (reference "H?") (unit 1) (value "MountingHole") (footprint "")
+    )
+    (path "/fc7e4fa4-6b96-4978-97ed-2756b031b2a0"
+      (reference "H?") (unit 1) (value "MountingHole") (footprint "")
+    )
     (path "/c4127e5f-30ba-43b1-b955-4e58698ee398"

Commit message: fix footprints
Parts:
- removed A1: Arduino_UNO_R3, Module:Arduino_Nano, symbol MCU_Module:Arduino_UNO_R3
- removed J29: Conn_02x06_Counter_Clockwise, symbol Connector_Generic:Conn_02x06_Counter_Clockwise
- added A1: Arduino_Nano_v3.x, Module:Arduino_Nano, symbol MCU_Module:Arduino_Nano_v3.x
- added AIN_5, AIN_6: Conn_01x02, Connector_Molex:Molex_Mini-Fit_Jr_5566-02A_2x01_P4.20mm_Vertical, symbol Connector_Generic:Conn_01x02
- added J29: Conn_02x05_Counter_Clockwise, Connector_Molex:Molex_Mini-Fit_Jr_5566-10A_2x05_P4.20mm_Vertical, symbol Connector_Generic:Conn_02x05_Counter_Clockwise
- added J30: Conn_01x01_Male, Connector_PinHeader_2.54mm:PinHeader_1x01_P2.54mm_Vertical, symbol Connector:Conn_01x01_Male
- added RAIN5, RAIN6: 10K, Resistor_SMD:R_1206_3216Metric, symbol Device:R
- 1WIRE1, 1WIRE2, 1WIRE3, DHT_1, DHT_2, I2C-1, I2C-2, I2C-3: footprint (none) -> Connector_Molex:Molex_Mini-Fit_Jr_5566-04A_2x02_P4.20mm_Vertical
- AIN_1, AIN_2, AIN_3, AIN_4: footprint (none) -> Connector_Molex:Molex_Mini-Fit_Jr_5566-02A_2x01_P4.20mm_Vertical
- FL1: footprint (none) -> Chinese_emi_filter:ChinezeFilter
- H1, H2, H3, H4: renamed from H?; footprint (none) -> MountingHole:MountingHole_3.2mm_M3_Pad
- K1, K2, K3, K4, K5, K6: footprint Relay_THT:Relay_SPDT_Omron-G5Q-1 -> Relay_THT:Relay_SPDT_Finder_36.11
- PS1, PS2: footprint Converter_ACDC:Converter_ACDC_Vigortronix_VTX-214-010-xxx_THT -> Converter_ACDC:Converter_ACDC_MeanWell_IRM-03-xx_THT
- renumbered D8 to DR1, D9 to DR2, D10 to DR3, D11 to DR4, D14 to DR5, D15 to DR6, U6 to U5, U7 to U6, U5 to UMAX1
Connections:
- net +12VA: now also A1.30 (VIN)
- net 1WIRE_DATA: now also A1.11 (D8)
- net 5VA: now also A1.27 (+5V), RAIN5.2, RAIN6.2
- net AIN1: now also A1.19 (A0)
- net AIN2: now also A1.20 (A1)
- net AIN3: now also A1.21 (A2)
- net AIN4: now also A1.22 (A3)
- net Ch1_Output: now also J29.3 (Pin_3)
- net Ch2_Output: now also J29.4 (Pin_4)
- net Ch3_Output: now also J29.5 (Pin_5)
- net Ch4_Output: now also J29.6 (Pin_6)
- net Ch5_Output: now also J29.7 (Pin_7)
- net Ch6_Output: now also J29.8 (Pin_8)
- net DHT1: now also A1.15 (D12)
- net DHT2: now also A1.16 (D13)
- net GND2: now also A1.29 (GND), AIN_5.2 (Pin_2), AIN_6.2 (Pin_2)
- net IN1: now also A1.5 (D2)
- net IN2: now also A1.6 (D3)
- net IN3: now also A1.7 (D4)
- net IN4: now also A1.8 (D5)
- net IN5: now also A1.9 (D6)
- net IN6: now also A1.10 (D7)
- net LINE: now also FL1.4, J29.1 (Pin_1); no longer FL1.1
- net Led1_in: now also J29.9 (Pin_9)
- net NEUT: now also FL1.2, J29.2 (Pin_2); no longer FL1.3
- net RX: now also A1.12 (D9)
- net Reset_in: now also J29.10 (Pin_10)
- net SCL: now also A1.24 (A5)
- net SDA: now also A1.23 (A4)
- net TX: now also A1.13 (D10)
- net T/R: now also A1.14 (D11)
- net AIN5: now reaches J27.1 (Pin_1)
- net AIN5: now also A1.25 (A6), AIN_5.1 (Pin_1), RAIN5.1
- net at PS1.1 (L), PS2.1 (L): now also FL1.3; no longer FL1.2
- net at PS1.2 (N), PS2.2 (N): now also FL1.1; no longer FL1.4
- net at J14.1 (Pin_1): now also A1.4 (GND)
- net at J26.1 (Pin_1): now also A1.28 (~{RESET})
- net at J15.1 (Pin_1): now also A1.17 (3V3)
- net at J28.1 (Pin_1): now also A1.18 (AREF)
- new net AIN6: A1.26 (A7), AIN_6.1 (Pin_1), J30.1 (Pin_1), RAIN6.1
- no-connect marks 6 -> 3
Other:
- note added: "IT IS NOT REAL FILTER"
- moved on the sheet: FL1

Commit message: step 2
Parts:
- removed J1, J10, J11, J12, J13, J14, J15, J16, J17, J2, J20, J21, J22, J23, J24, J25, J26, J27, J28, J3, J30, J4, J5, J6, J7, J8, J9: Conn_01x01_Male, Connector_PinHeader_2.54mm:PinHeader_1x01_P2.54mm_Vertical, symbol Connector:Conn_01x01_Male
- added J5v1, Jgnd1: Conn_01x05_Female, Connector_PinSocket_2.54mm:PinSocket_1x05_P2.54mm_Vertical, symbol Connector:Conn_01x05_Female
- added Ja1, Ja2: Conn_01x12_Male, Connector_PinSocket_2.54mm:PinSocket_1x12_P2.54mm_Vertical, symbol Connector:Conn_01x12_Male
- K1, K2, K3, K4, K5, K6: footprint Relay_THT:Relay_SPDT_Finder_36.11 -> Chinese_emi_filter:Relay_T75
- PS1, PS2: footprint Converter_ACDC:Converter_ACDC_MeanWell_IRM-03-xx_THT -> Chinese_emi_filter:Converter_ACDC_MeanWell_IRM-03-xx_THT
- SW1: footprint Resistor_SMD:R_1206_3216Metric -> Connector_PinHeader_2.54mm:PinHeader_1x02_P2.54mm_Vertical
- renumbered D3 to DRR1, D4 to DRR2, D5 to DRR3, D6 to DRR4, D12 to DRR5, D13 to DRR6, R1 to RR1, R8 to RR2, R9 to RR3, R10 to RR4, R20 to RR5, R21 to RR6, R2 to RRR1, R13 to RRR2, R14 to RRR3, R15 to RRR4, R22 to RRR5, R23 to RRR6
Connections:
- net 1WIRE_DATA: now also Ja1.6 (Pin_6)
- net 5VA: now also J5v1.1 (Pin_1), J5v1.2 (Pin_2), J5v1.3 (Pin_3), J5v1.4 (Pin_4), J5v1.5 (Pin_5), Ja2.2 (Pin_2)
- net AIN1: now also Ja2.5 (Pin_5)
- net AIN2: now also Ja2.6 (Pin_6)
- net AIN3: now also Ja2.7 (Pin_7)
- net AIN4: now also Ja2.8 (Pin_8)
- net AIN5: now also Ja2.11 (Pin_11)
- net AIN6: now also Ja2.12 (Pin_12)
- net DHT1: now also Ja1.2 (Pin_2)
- net DHT2: now also Ja1.1 (Pin_1)
- net GND2: now also A1.4 (GND), Jgnd1.1 (Pin_1), Jgnd1.2 (Pin_2), Jgnd1.3 (Pin_3), Jgnd1.4 (Pin_4), Jgnd1.5 (Pin_5)
- net IN1: now also Ja1.12 (Pin_12)
- net IN2: now also Ja1.11 (Pin_11)
- net IN3: now also Ja1.10 (Pin_10)
- net IN4: now also Ja1.9 (Pin_9)
- net IN5: now also Ja1.8 (Pin_8)
- net IN6: now also Ja1.7 (Pin_7)
- net RX: now also Ja1.5 (Pin_5)
- net SCL: now also Ja2.10 (Pin_10)
- net SDA: now also Ja2.9 (Pin_9)
- net TX: now also Ja1.4 (Pin_4)
- net T/R: now also Ja1.3 (Pin_3)
- net 3V3: now reaches A1.17 (3V3)
- net 3V3: now also Ja2.1 (Pin_1)
- net AREF: now reaches A1.18 (AREF)
- net AREF: now also Ja2.3 (Pin_3)
- net RESET: now reaches A1.28 (~{RESET})
- net RESET: now also Ja2.4 (Pin_4)

Commit message: v1 of pcb
Connections:
- net Ch1_Output is gone; now on net  Ch1_Output: J29.3 (Pin_3)
- net Ch2_Output is gone; now on net  Ch2_Output: J29.4 (Pin_4)
- net Ch3_Output is gone; now on net  Ch3_Output: J29.5 (Pin_5)
- net Ch4_Output is gone; now on net  Ch4_Output: J29.6 (Pin_6)
- net Ch5_Output is gone; now on net  Ch5_Output: J29.7 (Pin_7)
- net Ch6_Output is gone; now on net  Ch6_Output: J29.8 (Pin_8)
Changed lines of the file:
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@@
     (stroke (width 0) (type default) (color 0 0 0 0))
   )
-  (wire (pts (xy 208.28 90.17) (xy 215.9 90.17))
+  (wire (pts (xy 208.28 90.17) (xy 226.06 90.17))
     (stroke (width 0) (type default) (color 0 0 0 0))
   )
@@
     )
   )
+  (global_label " Ch5_Output" (shape input) (at 289.56 186.69 0) (fields_autoplaced)
+    (effects (font (size 1.27 1.27)) (justify left))
+    (property "Intersheet References" "${INTERSHEET_REFS}" (id 0) (at 303.766 186.6106 0)
+      (effects (font (size 1.27 1.27)) (justify left) hide)
+    )
+  )
   (global_label "5VA" (shape output) (at 129.54 198.12 0) (fields_autoplaced)
     (effects (font (size 1.27 1.27)) (justify left))
@@
     )
   )
-  (global_label "Ch6_Output" (shape input) (at 289.56 184.15 0) (fields_autoplaced)
-    (effects (font (size 1.27 1.27)) (justify left))
-    (property "Intersheet References" "${INTERSHEET_REFS}" (id 0) (at 302.7983 184.0706 0)
-      (effects (font (size 1.27 1.27)) (justify left) hide)
-    )
-  )
   (global_label "IN4" (shape input) (at 125.73 129.54 180) (fields_autoplaced)
     (effects (font (size 1.27 1.27)) (justify right))
@@
     )
   )
-  (global_label " Ch1_Output" (shape output) (at 215.9 22.86 0) (fields_autoplaced)
+  (global_label " Ch1_Output" (shape input) (at 215.9 22.86 0) (fields_autoplaced)
     (effects (font (size 1.27 1.27)) (justify left))
     (property "Intersheet References" "${INTERSHEET_REFS}" (id 0) (at 230.106 22.7806 0)
@@
     )
   )
-  (global_label " Ch4_Output" (shape output) (at 217.17 121.92 0) (fields_autoplaced)
+  (global_label " Ch4_Output" (shape input) (at 217.17 121.92 0) (fields_autoplaced)
     (effects (font (size 1.27 1.27)) (justify left))
     (property "Intersheet References" "${INTERSHEET_REFS}" (id 0) (at 231.376 121.8406 0)
@@
     )
   )
-  (global_label "Ch5_Output" (shape input) (at 289.56 186.69 0) (fields_autoplaced)
-    (effects (font (size 1.27 1.27)) (justify left))
-    (property "Intersheet References" "${INTERSHEET_REFS}" (id 0) (at 302.7983 186.6106 0)
-      (effects (font (size 1.27 1.27)) (justify left) hide)
-    )
-  )
   (global_label "AIN6" (shape input) (at 83.82 134.62 0) (fields_autoplaced)
     (effects (font (size 1.27 1.27)) (justify left))
@@
     )
   )
-  (global_label " Ch3_Output" (shape output) (at 215.9 90.17 0) (fields_autoplaced)
-    (effects (font (size 1.27 1.27)) (justify left))
-    (property "Intersheet References" "${INTERSHEET_REFS}" (id 0) (at 230.106 90.0906 0)
+  (global_label " Ch3_Output" (shape input) (at 226.06 90.17 0) (fields_autoplaced)
+    (effects (font (size 1.27 1.27)) (justify left))
+    (property "Intersheet References" "${INTERSHEET_REFS}" (id 0) (at 240.266 90.0906 0)
       (effects (font (size 1.27 1.27)) (justify left) hide)
     )
@@
     )
   )
+  (global_label " Ch3_Output" (shape input) (at 273.05 190.5 180) (fields_autoplaced)
+    (effects (font (size 1.27 1.27)) (justify right))
+    (property "Intersheet References" "${INTERSHEET_REFS}" (id 0) (at 258.844 190.5794 0)
+      (effects (font (size 1.27 1.27)) (justify right) hide)
+    )
+  )
   (global_label "5VA" (shape output) (at 223.52 240.03 0) (fields_autoplaced)
     (effects (font (size 1.27 1.27)) (justify left))
@@
     )
   )
-  (global_label " Ch2_Output" (shape output) (at 215.9 57.15 0) (fields_autoplaced)
+  (global_label " Ch2_Output" (shape input) (at 215.9 57.15 0) (fields_autoplaced)
     (effects (font (size 1.27 1.27)) (justify left))
     (property "Intersheet References" "${INTERSHEET_REFS}" (id 0) (at 230.106 57.0706 0)
@@
     )
   )
-  (global_label " Ch6_Output" (shape output) (at 353.06 57.15 0) (fields_autoplaced)
+  (global_label " Ch6_Output" (shape input) (at 353.06 57.15 0) (fields_autoplaced)
     (effects (font (size 1.27 1.27)) (justify left))
     (property "Intersheet References" "${INTERSHEET_REFS}" (id 0) (at 367.266 57.0706 0)
@@
     )
   )
-  (global_label "Ch1_Output" (shape input) (at 273.05 185.42 180) (fields_autoplaced)
-    (effects (font (size 1.27 1.27)) (justify right))
-    (property "Intersheet References" "${INTERSHEET_REFS}" (id 0) (at 259.8117 185.3406 0)
-      (effects (font (size 1.27 1.27)) (justify right) hide)
-    )
-  )
-  (global_label "Ch3_Output" (shape input) (at 273.05 190.5 180) (fields_autoplaced)
-    (effects (font (size 1.27 1.27)) (justify right))
-    (property "Intersheet References" "${INTERSHEET_REFS}" (id 0) (at 259.8117 190.4206 0)
-      (effects (font (size 1.27 1.27)) (justify right) hide)
-    )
-  )
   (global_label "AIN2" (shape input) (at 83.82 119.38 0) (fields_autoplaced)
     (effects (font (size 1.27 1.27)) (justify left))
@@
     )
   )
+  (global_label " Ch1_Output" (shape input) (at 273.05 185.42 180) (fields_autoplaced)
+    (effects (font (size 1.27 1.27)) (justify right))
+    (property "Intersheet References" "${INTERSHEET_REFS}" (id 0) (at 258.844 185.4994 0)
+      (effects (font (size 1.27 1.27)) (justify right) hide)
+    )
+  )
   (global_label "5VA" (shape input) (at 298.45 214.63 180) (fields_autoplaced)
     (effects (font (size 1.27 1.27)) (justify right))
@@
     )
   )
+  (global_label " Ch4_Output" (shape input) (at 289.56 189.23 0) (fields_autoplaced)
+    (effects (font (size 1.27 1.27)) (justify left))
+    (property "Intersheet References" "${INTERSHEET_REFS}" (id 0) (at 303.766 189.1506 0)
+      (effects (font (size 1.27 1.27)) (justify left) hide)
+    )
+  )
   (global_label "3V3" (shape input) (at 388.62 153.67 180) (fields_autoplaced)
     (effects (font (size 1.27 1.27)) (justify right))
@@
     )
   )
+  (global_label " Ch2_Output" (shape input) (at 273.05 187.96 180) (fields_autoplaced)
+    (effects (font (size 1.27 1.27)) (justify right))
+    (property "Intersheet References" "${INTERSHEET_REFS}" (id 0) (at 258.844 188.0394 0)
+      (effects (font (size 1.27 1.27)) (justify right) hide)
+    )
+  )
   (global_label "IN2" (shape input) (at 124.46 64.77 180) (fields_autoplaced)
     (effects (font (size 1.27 1.27)) (justify right))
@@
     )
   )
-  (global_label "Ch2_Output" (shape input) (at 273.05 187.96 180) (fields_autoplaced)
-    (effects (font (size 1.27 1.27)) (justify right))
-    (property "Intersheet References" "${INTERSHEET_REFS}" (id 0) (at 259.8117 187.8806 0)
-      (effects (font (size 1.27 1.27)) (justify right) hide)
-    )
-  )
   (global_label "DHT1" (shape input) (at 368.3 151.13 180) (fields_autoplaced)
     (effects (font (size 1.27 1.27)) (justify right))
@@
     )
   )
-  (global_label "Ch4_Output" (shape input) (at 289.56 189.23 0) (fields_autoplaced)
-    (effects (font (size 1.27 1.27)) (justify left))
-    (property "Intersheet References" "${INTERSHEET_REFS}" (id 0) (at 302.7983 189.3094 0)
-      (effects (font (size 1.27 1.27)) (justify left) hide)
-    )
-  )
-  (global_label " Ch5_Output" (shape output) (at 351.79 25.4 0) (fields_autoplaced)
+  (global_label " Ch5_Output" (shape input) (at 351.79 25.4 0) (fields_autoplaced)
     (effects (font (size 1.27 1.27)) (justify left))
     (property "Intersheet References" "${INTERSHEET_REFS}" (id 0) (at 365.996 25.3206 0)
       (effects (font (size 1.27 1.27)) (justify left) hide)
     )
+  )
+  (global_label " Ch6_Output" (shape input) (at 289.56 184.15 0) (fields_autoplaced)
+    (effects (font (size 1.27 1.27)) (justify left))
+    (property "Intersheet References" "${INTERSHEET_REFS}" (id 0) (at 303.766 184.0706 0)
+      (effects (font (size 1.27 1.27)) (justify left) hide)
+    )

Commit message: added 4 layers struct
Parts:
- added rel1-NO1, rel2-NO1, rel3-NO1, rel4-NO1, rel5-NO1, rel6-NO1: Conn_01x01_Male, Connector_PinHeader_2.54mm:PinHeader_1x01_P2.54mm_Vertical, symbol Connector:Conn_01x01_Male
- renumbered rel1-2 to rel1-NC1, rel2-2 to rel2-NC1, rel3-2 to rel3-NC1, rel4-2 to rel4-NC1, rel5-2 to rel5-NC1, rel6-2 to rel6-NC1
Connections:
- net  Ch1_Output: now also rel1-NO1.1 (Pin_1)
- net  Ch2_Output: now also rel2-NO1.1 (Pin_1)
- net  Ch3_Output: now also rel3-NO1.1 (Pin_1)
- net  Ch4_Output: now also rel4-NO1.1 (Pin_1)
- net  Ch5_Output: now also rel5-NO1.1 (Pin_1)
- net  Ch6_Output: now also rel6-NO1.1 (Pin_1)
