File: kolos_system_2022.kicad_sch (KiCad schematic)
At the start: 112 parts, among them J18 8P8C_LED, J19 8P8C_LED, J29 Conn_02x05_Counter_Clockwise, J5v1 Conn_01x05_Female, K1 G5Q-1, K2 G5Q-1, K3 G5Q-1, K4 G5Q-1, K5 G5Q-1, K6 G5Q-1, Q1 BC848W, Q2 BC848W, Q3 BC848W, Q4 BC848W, Q5 BC848W, Q6 BC848W, SW1 SW_DIP_x01, U1 EL817, U2 EL817, U3 EL817, U4 EL817, U5 EL817, U6 EL817

Commit message: prepared to manufacturing
Parts:
- added J1, J2: Conn_01x01_Male, Connector_PinHeader_2.54mm:PinHeader_1x01_P2.54mm_Vertical, symbol Connector:Conn_01x01_Male
Connections:
- net Led1_in: now also J1.1 (Pin_1)
- net Reset_in: now also J2.1 (Pin_1)
Changed lines of the file:
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@@
     )
   )
+  (global_label "Led1_in" (shape input) (at 311.15 167.64 0) (fields_autoplaced)
+    (effects (font (size 1.27 1.27)) (justify left))
+    (property "Intersheet References" "${INTERSHEET_REFS}" (id 0) (at 320.7598 167.7194 0)
+      (effects (font (size 1.27 1.27)) (justify left) hide)
+    )
+  )
   (global_label "SCL" (shape input) (at 388.62 130.81 180) (fields_autoplaced)
     (effects (font (size 1.27 1.27)) (justify right))
@@
     )
   )
+  (global_label "Reset_in" (shape input) (at 311.15 171.45 0) (fields_autoplaced)
+    (effects (font (size 1.27 1.27)) (justify left))
+    (property "Intersheet References" "${INTERSHEET_REFS}" (id 0) (at 321.4855 171.5294 0)
+      (effects (font (size 1.27 1.27)) (justify left) hide)
+    )
+  )
   (global_label "SDA" (shape input) (at 262.89 212.09 180) (fields_autoplaced)
     (effects (font (size 1.27 1.27)) (justify right))
@@
     (pin "2")
   )
+  (symbol (lib_id "Connector:Conn_01x01_Male") (at 306.07 167.64 0) (unit 1)
+    (in_bom yes) (on_board yes) (fields_autoplaced)
+    (property "Reference" "J1" (id 0) (at 306.705 165.1 0))
+    (property "Value" "Conn_01x01_Male" (id 1) (at 306.705 165.1 0)
+      (effects (font (size 1.27 1.27)) hide)
+    )
+    (property "Footprint" "Connector_PinHeader_2.54mm:PinHeader_1x01_P2.54mm_Vertical" (id 2) (at 306.07 167.64 0)
+      (effects (font (size 1.27 1.27)) hide)
+    )
+    (property "Datasheet" "~" (id 3) (at 306.07 167.64 0)
+      (effects (font (size 1.27 1.27)) hide)
+    )
+    (pin "1")
+  )
   (symbol (lib_id "Device:R") (at 163.83 187.96 90) (unit 1)
     (in_bom yes) (on_board yes)
@@
     (pin "2")
   )
+  (symbol (lib_id "Connector:Conn_01x01_Male") (at 306.07 171.45 0) (unit 1)
+    (in_bom yes) (on_board yes) (fields_autoplaced)
+    (property "Reference" "J2" (id 0) (at 306.705 166.37 0))
+    (property "Value" "Conn_01x01_Male" (id 1) (at 306.705 168.91 0)
+      (effects (font (size 1.27 1.27)) hide)
+    )
+    (property "Footprint" "Connector_PinHeader_2.54mm:PinHeader_1x01_P2.54mm_Vertical" (id 2) (at 306.07 171.45 0)
+      (effects (font (size 1.27 1.27)) hide)
+    )
+    (property "Datasheet" "~" (id 3) (at 306.07 171.45 0)
+      (effects (font (size 1.27 1.27)) hide)
+    )
+    (pin "1")
+  )
   (symbol (lib_id "Connector:Conn_01x01_Male") (at 345.44 53.34 180) (unit 1)
     (in_bom yes) (on_board yes) (fields_autoplaced)
@@
       (reference "I2C-3") (unit 1) (value "Conn_01x04") (footprint "Connector_Molex:Molex_Mini-Fit_Jr_5566-04A_2x02_P4.20mm_Vertical")
     )
+    (path "/2ef0e97d-70a0-4db7-b378-ebd1da6d1fac"
+      (reference "J1") (unit 1) (value "Conn_01x01_Male") (footprint "Connector_PinHeader_2.54mm:PinHeader_1x01_P2.54mm_Vertical")
+    )
+    (path "/c9d2d0e8-69ee-4eb5-92fc-a6f3749a34e3"
+      (reference "J2") (unit 1) (value "Conn_01x01_Male") (footprint "Connector_PinHeader_2.54mm:PinHeader_1x01_P2.54mm_Vertical")
+    )
     (path "/d9e438eb-6a30-4ee6-9093-110527e75662"
