File: kolos_system_2022.kicad_sch (KiCad schematic)
At the start: 112 parts, among them J18 8P8C_LED, J19 8P8C_LED, J29 Conn_02x05_Counter_Clockwise, J5v1 Conn_01x05_Female, K1 G5Q-1, K2 G5Q-1, K3 G5Q-1, K4 G5Q-1, K5 G5Q-1, K6 G5Q-1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

Commit message: second version of pcb
Parts:
- added J1, J2: Conn_01x01_Male, Connector_PinHeader_2.54mm:PinHeader_1x01_P2.54mm_Vertical, symbol Connector:Conn_01x01_Male
Connections:
- net Led1_in: now also J2.1 (Pin_1)
- net Reset_in: now also J1.1 (Pin_1)
Changed lines of the file:
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@@
     )
   )
+  (global_label "Reset_in" (shape input) (at 314.96 167.64 0) (fields_autoplaced)
+    (effects (font (size 1.27 1.27)) (justify left))
+    (property "Intersheet References" "${INTERSHEET_REFS}" (id 0) (at 325.2955 167.7194 0)
+      (effects (font (size 1.27 1.27)) (justify left) hide)
+    )
+  )
   (global_label "AIN1" (shape input) (at 340.36 171.45 180) (fields_autoplaced)
     (effects (font (size 1.27 1.27)) (justify right))
@@
     )
   )
+  (global_label "Led1_in" (shape input) (at 314.96 172.72 0) (fields_autoplaced)
+    (effects (font (size 1.27 1.27)) (justify left))
+    (property "Intersheet References" "${INTERSHEET_REFS}" (id 0) (at 324.5698 172.7994 0)
+      (effects (font (size 1.27 1.27)) (justify left) hide)
+    )
+  )
   (global_label "5VA" (shape input) (at 298.45 214.63 180) (fields_autoplaced)
     (effects (font (size 1.27 1.27)) (justify right))
@@
     (pin "2")
   )
+  (symbol (lib_id "Connector:Conn_01x01_Male") (at 309.88 172.72 0) (unit 1)
+    (in_bom yes) (on_board yes) (fields_autoplaced)
+    (property "Reference" "J2" (id 0) (at 310.515 167.64 0))
+    (property "Value" "Conn_01x01_Male" (id 1) (at 310.515 170.18 0))
+    (property "Footprint" "Connector_PinHeader_2.54mm:PinHeader_1x01_P2.54mm_Vertical" (id 2) (at 309.88 172.72 0)
+      (effects (font (size 1.27 1.27)) hide)
+    )
+    (property "Datasheet" "~" (id 3) (at 309.88 172.72 0)
+      (effects (font (size 1.27 1.27)) hide)
+    )
+    (pin "1")
+  )
   (symbol (lib_id "power:GND2") (at 375.92 191.77 0) (unit 1)
     (in_bom yes) (on_board yes) (fields_autoplaced)
@@
     (pin "1")
   )
+  (symbol (lib_id "Connector:Conn_01x01_Male") (at 309.88 167.64 0) (unit 1)
+    (in_bom yes) (on_board yes) (fields_autoplaced)
+    (property "Reference" "J1" (id 0) (at 310.515 162.56 0))
+    (property "Value" "Conn_01x01_Male" (id 1) (at 310.515 165.1 0))
+    (property "Footprint" "Connector_PinHeader_2.54mm:PinHeader_1x01_P2.54mm_Vertical" (id 2) (at 309.88 167.64 0)
+      (effects (font (size 1.27 1.27)) hide)
+    )
+    (property "Datasheet" "~" (id 3) (at 309.88 167.64 0)
+      (effects (font (size 1.27 1.27)) hide)
+    )
+    (pin "1")
+  )
   (symbol (lib_id "Mechanical:MountingHole") (at 391.16 228.6 0) (unit 1)
     (in_bom yes) (on_board yes) (fields_autoplaced)
@@
       (reference "I2C-3") (unit 1) (value "Conn_01x04") (footprint "Connector_Molex:Molex_Mini-Fit_Jr_5566-04A_2x02_P4.20mm_Vertical")
     )
+    (path "/fa21e2f7-d34d-43aa-912c-a5e81ffcf9a4"
+      (reference "J1") (unit 1) (value "Conn_01x01_Male") (footprint "Connector_PinHeader_2.54mm:PinHeader_1x01_P2.54mm_Vertical")
+    )
+    (path "/0d995815-0174-46af-9a65-98edd7e158d0"
+      (reference "J2") (unit 1) (value "Conn_01x01_Male") (footprint "Connector_PinHeader_2.54mm:PinHeader_1x01_P2.54mm_Vertical")
+    )
     (path "/d9e438eb-6a30-4ee6-9093-110527e75662"
